File: D1_PCB/D1_PCB/D1_PCB.kicad_pcb (KiCad board)
At the start: 2 copper layers, 86.4 x 45.7 mm, 12 parts, among them J1 BB_RIGHT, J2 BB_LEFT, J3 Conn_01x02, J4 Conn_01x02

Commit message: Utility D1 PCB changes
Parts:
- added 5V1: Conn_01x04_Pin, Connector_PinHeader_2.54mm:PinHeader_1x04_P2.54mm_Vertical, F.Cu at (182.9, 85.1)
- added C2: 2.2uF, Capacitor_THT:C_Disc_D3.0mm_W2.0mm_P2.50mm, F.Cu at (184.2, 96.5)
- added G***: LOGO, Lumensalis:LSLogo1, F.Cu at (185.4, 127.0)
- added G***: LOGO, Lumensalis:LSLogo1, B.Cu at (184.2, 115.6)
- added GND1: Conn_01x04_Pin, Connector_PinHeader_2.54mm:PinHeader_1x04_P2.54mm_Vertical, F.Cu at (188.0, 85.1)
- added J5: Conn_01x04_Pin, Connector_PinHeader_2.54mm:PinHeader_1x04_P2.54mm_Vertical, F.Cu at (123.2, 129.5)
- added JLGND1: SolderJumper_2_Bridged, Jumper:SolderJumper-2_P1.3mm_Bridged2Bar_RoundedPad1.0x1.5mm, F.Cu at (178.4, 87.6)
- added JLVDD1: SolderJumper_2_Bridged, Jumper:SolderJumper-2_P1.3mm_Bridged2Bar_RoundedPad1.0x1.5mm, F.Cu at (178.4, 91.4)
- added JNXA1: SolderJumper_2_Bridged, Jumper:SolderJumper-2_P1.3mm_Bridged2Bar_RoundedPad1.0x1.5mm, F.Cu at (152.4, 92.7)
- added JNXB1: SolderJumper_2_Bridged, Jumper:SolderJumper-2_P1.3mm_Bridged2Bar_RoundedPad1.0x1.5mm, F.Cu at (162.6, 92.7)
- added JNXC2: SolderJumper_2_Bridged, Jumper:SolderJumper-2_P1.3mm_Bridged2Bar_RoundedPad1.0x1.5mm, F.Cu at (172.7, 92.7)
- added NeoXA1: Conn_01x03_MountingPin, Connector_JST:JST_GH_SM03B-GHS-TB_1x03-1MP_P1.25mm_Horizontal, F.Cu at (153.7, 83.9)
- added NeoXB1: Conn_01x03_MountingPin, Connector_JST:JST_GH_SM03B-GHS-TB_1x03-1MP_P1.25mm_Horizontal, F.Cu at (162.6, 83.8)
- added NeoXC2: Conn_01x03_MountingPin, Connector_JST:JST_GH_SM03B-GHS-TB_1x03-1MP_P1.25mm_Horizontal, F.Cu at (171.5, 83.9)
- added QwiicA1: Conn_01x04_MountingPin, Connector_JST:JST_SH_SM04B-SRSS-TB_1x04-1MP_P1.00mm_Horizontal, F.Cu at (135.7, 84.5)
- added QwiicB1: Conn_01x04_MountingPin, Connector_JST:JST_SH_SM04B-SRSS-TB_1x04-1MP_P1.00mm_Horizontal, F.Cu at (124.2, 84.4)
- added R1: 4K7, Resistor_THT:R_Axial_DIN0204_L3.6mm_D1.6mm_P2.54mm_Vertical, F.Cu at (125.7, 92.7)
- added R2: 4K7, Resistor_THT:R_Axial_DIN0204_L3.6mm_D1.6mm_P2.54mm_Vertical, F.Cu at (119.4, 90.2)
- added R3: 4K7, Resistor_THT:R_Axial_DIN0204_L3.6mm_D1.6mm_P2.54mm_Vertical, F.Cu at (129.5, 90.2)
- added R4: 4K7, Resistor_THT:R_Axial_DIN0204_L3.6mm_D1.6mm_P2.54mm_Vertical, F.Cu at (138.4, 92.7)
- added REF**: MountingHole_2.2mm_M2_Pad, MountingHole:MountingHole_2.2mm_M2_Pad, F.Cu at (114.3, 82.5)
- added REF**: MountingHole_2.2mm_M2_Pad, MountingHole:MountingHole_2.2mm_M2_Pad, F.Cu at (199.4, 82.5)
- added REF**: MountingHole_2.2mm_M2_Pad, MountingHole:MountingHole_2.2mm_M2_Pad, F.Cu at (199.4, 130.8)
- added REF**: MountingHole_2.2mm_M2_Pad, MountingHole:MountingHole_2.2mm_M2_Pad, F.Cu at (114.3, 130.8)
- added SCL_A1: SolderJumper_2_Bridged, Jumper:SolderJumper-2_P1.3mm_Bridged2Bar_RoundedPad1.0x1.5mm, F.Cu at (133.3, 95.2)
- added SCL_B1: SolderJumper_2_Bridged, Jumper:SolderJumper-2_P1.3mm_Bridged2Bar_RoundedPad1.0x1.5mm, F.Cu at (121.9, 95.2)
- added SDA_A1: SolderJumper_2_Bridged, Jumper:SolderJumper-2_P1.3mm_Bridged2Bar_RoundedPad1.0x1.5mm, F.Cu at (135.9, 95.2)
- added SDA_B1: SolderJumper_2_Bridged, Jumper:SolderJumper-2_P1.3mm_Bridged2Bar_RoundedPad1.0x1.5mm, F.Cu at (124.4, 95.2)
- added c3v3: Conn_01x04_Pin, Connector_PinHeader_2.54mm:PinHeader_1x04_P2.54mm_Vertical, B.Cu at (193.0, 85.1)
- added t3v3: TestPoint, Connector_Pin:Pin_D1.3mm_L11.0mm, F.Cu at (162.6, 123.2)
- added t5V1: TestPoint, Connector_Pin:Pin_D1.3mm_L11.0mm, F.Cu at (143.5, 120.7)
- added tGND1: TestPoint, Connector_Pin:Pin_D1.3mm_L11.0mm, F.Cu at (143.5, 115.6)
- moved J3 0.28 mm to (132.1, 121.9)
Connections:
- J3 pad 1: unconnected-(J3-Pin_1-Pad1) -> Net-(J3-Pin_1)
- J3 pad 2: unconnected-(J3-Pin_2-Pad2) -> Net-(J3-Pin_2)
- J4 pad 1: unconnected-(J4-Pin_1-Pad1) -> Net-(J4-Pin_1)
- J4 pad 2: unconnected-(J4-Pin_2-Pad2) -> Net-(J4-Pin_2)
Routing:
- net D1M_GND: track 98.1 -> 358.0 mm, vias 0 -> 20
- net D1M_3V3: track 43.4 -> 208.9 mm, vias 0 -> 4
- net D1M_VDD: track 75.9 -> 143.1 mm, vias 0 -> 1
- net SML_7: track 6.13 -> 65.9 mm
- net SML_6: track 14.8 -> 53.5 mm
- net LEDVIN: track 0.00 -> 38.6 mm, vias 0 -> 4
- net LEDGND: track 0.00 -> 33.2 mm, vias 0 -> 3
- net Net-(J4-Pin_1): track 0.00 -> 29.8 mm, vias 0 -> 2
- net SML_5: track 14.8 -> 43.5 mm
- net Net-(J4-Pin_2): track 0.00 -> 26.2 mm, vias 0 -> 2
- net D1M_D2: track 63.3 -> 81.5 mm
- net D1M_D1: track 60.3 -> 77.5 mm
- net SML_4: track 14.8 -> 30.5 mm
- net Net-(J3-Pin_1): track 0.00 -> 13.7 mm
- net SML_3: track 14.8 -> 28.4 mm
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Other:
- board size 86.4 x 45.7 mm -> 92.7 x 55.9 mm
