File: D1_PCB/D1_PCB/D1_PCB.kicad_sch (KiCad schematic)
At the start: 13 parts, among them J1 BB_RIGHT, J2 BB_LEFT, J3 Conn_01x02, J4 Conn_01x02, U1 WEMOS_D1_mini

Commit message: Utility D1 PCB changes
Parts:
- added 5V1, GND1, J5, c3v3: Conn_01x04_Pin, Connector_PinHeader_2.54mm:PinHeader_1x04_P2.54mm_Vertical, symbol Connector:Conn_01x04_Pin
- added C2: 2.2uF, Capacitor_THT:C_Disc_D3.0mm_W2.0mm_P2.50mm, symbol Device:C
- added JLGND1, JLVDD1, JNXA1, JNXB1, JNXC2, SCL_A1, SCL_B1, SDA_A1, SDA_B1: SolderJumper_2_Bridged, Jumper:SolderJumper-2_P1.3mm_Bridged2Bar_RoundedPad1.0x1.5mm, symbol Jumper:SolderJumper_2_Bridged
- added NeoXA1, NeoXB1, NeoXC2: Conn_01x03_MountingPin, Connector_JST:JST_GH_SM03B-GHS-TB_1x03-1MP_P1.25mm_Horizontal, symbol Connector_Generic_MountingPin:Conn_01x03_MountingPin
- added QwiicA1, QwiicB1: Conn_01x04_MountingPin, Connector_JST:JST_SH_SM04B-SRSS-TB_1x04-1MP_P1.00mm_Horizontal, symbol Connector_Generic_MountingPin:Conn_01x04_MountingPin
- added R1, R2, R3, R4: 4K7, Resistor_THT:R_Axial_DIN0204_L3.6mm_D1.6mm_P2.54mm_Vertical, symbol Device:R_US
- added t3v3, t5V1, tGND1: TestPoint, Connector_Pin:Pin_D1.3mm_L11.0mm, symbol Connector:TestPoint
- U1: now not fitted
Connections:
- net +3V3: now also QwiicA1.2 (Pin_2), QwiicB1.2 (Pin_2), R1.1, R2.1, R3.1, R4.1, c3v3.1 (Pin_1), c3v3.2 (Pin_2), c3v3.3 (Pin_3), c3v3.4 (Pin_4), t3v3.1
- net +5VD: now also 5V1.1 (Pin_1), 5V1.2 (Pin_2), 5V1.3 (Pin_3), 5V1.4 (Pin_4), C2.1, JLVDD1.1 (A), t5V1.1
- net D1M_D1: now also SCL_A1.1 (A)
- net D1M_D2: now also SDA_A1.1 (A)
- net GND: now also C2.2, GND1.1 (Pin_1), GND1.2 (Pin_2), GND1.3 (Pin_3), GND1.4 (Pin_4), JLGND1.1 (A), NeoXA1.MP (MountPin), NeoXB1.MP (MountPin), NeoXC2.MP (MountPin), QwiicA1.1 (Pin_1), QwiicA1.MP (MountPin), QwiicB1.1 (Pin_1), QwiicB1.MP (MountPin), tGND1.1
- net SML_3: now also SDA_B1.1 (A)
- net SML_4: now also SCL_B1.1 (A)
- net SML_5: now also JNXA1.1 (A)
- net SML_6: now also JNXB1.1 (A)
- net SML_7: now also JNXC2.1 (A)
- net at J3.1 (Pin_1): now also J5.2 (Pin_2)
- net at J3.2 (Pin_2): now also J5.1 (Pin_1)
- net at J4.1 (Pin_1): now also J5.3 (Pin_3)
- net at J4.2 (Pin_2): now also J5.4 (Pin_4)
- new net LEDGND: JLGND1.2 (B), NeoXA1.1 (Pin_1), NeoXB1.1 (Pin_1), NeoXC2.1 (Pin_1)
- new net LEDVIN: JLVDD1.2 (B), NeoXA1.3 (Pin_3), NeoXB1.3 (Pin_3), NeoXC2.3 (Pin_3)
- new net NXA_DOUT: JNXA1.2 (B), NeoXA1.2 (Pin_2)
- new net NXB_DOUT: JNXB1.2 (B), NeoXB1.2 (Pin_2)
- new net NXC_DOUT: JNXC2.2 (B), NeoXC2.2 (Pin_2)
- new net QA_SCL: QwiicA1.4 (Pin_4), R3.2, SCL_A1.2 (B)
- new net QA_SDA: QwiicA1.3 (Pin_3), R4.2, SDA_A1.2 (B)
- new net QB_SCL: QwiicB1.4 (Pin_4), R2.2, SCL_B1.2 (B)
- new net QB_SDA: QwiicB1.3 (Pin_3), R1.2, SDA_B1.2 (B)
Other:
- moved on the sheet: J3, J4
